File: psu-12-5-0-12.sch (KiCad schematic (older format))
At the start: 20 parts, among them J1 12/0/12VAC, J2 12/5/0/-12VDC, U1 L7812, U2 L7912, U3 L7805

Commit message: Footprints.
Parts:
- C1, C2: footprint (none) -> Capacitor_THT:CP_Axial_L42.5mm_D20.0mm_P49.00mm_Horizontal
- C3: footprint (none) -> Capacitor_THT:C_Rect_L11.0mm_W4.2mm_P10.00mm_MKT
- C4, C6: footprint (none) -> Capacitor_THT:CP_Axial_L11.0mm_D5.0mm_P18.00mm_Horizontal
- C5, C8: footprint (none) -> Capacitor_THT:C_Rect_L9.0mm_W2.5mm_P7.50mm_MKT
- C7: footprint (none) -> Capacitor_THT:CP_Radial_Tantal_D6.0mm_P5.00mm
- D1: footprint (none) -> Diode_THT:Diode_Bridge_Vishay_KBU
- D2: footprint (none) -> LED_THT:LED_D5.0mm_FlatTop
- D3: footprint (none) -> Diode_THT:D_A-405_P10.16mm_Horizontal
- D4, D5: footprint (none) -> Diode_THT:D_A-405_P7.62mm_Horizontal
- J1: footprint (none) -> TerminalBlock:TerminalBlock_bornier-3_P5.08mm
- J2: footprint (none) -> TerminalBlock:TerminalBlock_bornier-4_P5.08mm
- R1: footprint (none) -> Package_TO_SOT_THT:TO-126-2_Vertical
- R2: footprint (none) -> Resistor_THT:R_Axial_DIN0207_L6.3mm_D2.5mm_P10.16mm_Horizontal
- U1, U2, U3: footprint (none) -> Package_TO_SOT_THT:TO-220-3_Vertical
Changed lines of the file:
@@
 F 0 "J1" H 1320 2675 50  0000 C CNN
 F 1 "12/0/12VAC" H 1320 2766 50  0000 C CNN
-F 2 "" H 1400 3000 50  0001 C CNN
+F 2 "TerminalBlock:TerminalBlock_bornier-3_P5.08mm" H 1400 3000 50  0001 C CNN
 F 3 "~" H 1400 3000 50  0001 C CNN
 	1    1400 3000
@@
 F 0 "D1" H 2500 3025 50  0000 L CNN
 F 1 "-AA+" H 2225 3225 50  0000 L CNN
-F 2 "" H 2350 3200 50  0001 C CNN
+F 2 "Diode_THT:Diode_Bridge_Vishay_KBU" H 2350 3200 50  0001 C CNN
 F 3 "~" H 2350 3200 50  0001 C CNN
 	1    2350 3200
@@
 F 0 "D2" V 2888 3433 50  0000 R CNN
 F 1 "LED" V 2797 3433 50  0000 R CNN
-F 2 "" H 2850 3550 50  0001 C CNN
+F 2 "LED_THT:LED_D5.0mm_FlatTop" H 2850 3550 50  0001 C CNN
 F 3 "~" H 2850 3550 50  0001 C CNN
 	1    2850 3550
@@
 F 0 "R2" H 2920 3146 50  0000 L CNN
 F 1 "3k9" H 2920 3055 50  0000 L CNN
-F 2 "" V 2780 3100 50  0001 C CNN
+F 2 "Resistor_THT:R_Axial_DIN0207_L6.3mm_D2.5mm_P10.16mm_Horizontal" V 2780 3100 50  0001 C CNN
 F 3 "~" H 2850 3100 50  0001 C CNN
 	1    2850 3100
@@
 F 0 "C3" H 3715 3146 50  0000 L CNN
 F 1 "330n" H 3715 3055 50  0000 L CNN
-F 2 "" H 3638 2950 50  0001 C CNN
+F 2 "Capacitor_THT:C_Rect_L11.0mm_W4.2mm_P10.00mm_MKT" H 3638 2950 50  0001 C CNN
 F 3 "~" H 3600 3100 50  0001 C CNN
 	1    3600 3100
@@
 F 0 "C8" H 6565 2746 50  0000 L CNN
 F 1 "100n" H 6565 2655 50  0000 L CNN
-F 2 "" H 6488 2550 50  0001 C CNN
+F 2 "Capacitor_THT:C_Rect_L9.0mm_W2.5mm_P7.50mm_MKT" H 6488 2550 50  0001 C CNN
 F 3 "~" H 6450 2700 50  0001 C CNN
 	1    6450 2700
@@
 F 0 "C5" H 4665 3146 50  0000 L CNN
 F 1 "100n" H 4665 3055 50  0000 L CNN
-F 2 "" H 4588 2950 50  0001 C CNN
+F 2 "Capacitor_THT:C_Rect_L9.0mm_W2.5mm_P7.50mm_MKT" H 4588 2950 50  0001 C CNN
 F 3 "~" H 4550 3100 50  0001 C CNN
 	1    4550 3100
@@
 F 0 "C1" H 3318 3146 50  0000 L CNN
 F 1 "4m7" H 3318 3055 50  0000 L CNN
-F 2 "" H 3238 2950 50  0001 C CNN
+F 2 "Capacitor_THT:CP_Axial_L42.5mm_D20.0mm_P49.00mm_Horizontal" H 3238 2950 50  0001 C CNN
 F 3 "~" H 3200 3100 50  0001 C CNN
 	1    3200 3100
@@
 F 0 "C2" H 3318 3596 50  0000 L CNN
 F 1 "4m7" H 3318 3505 50  0000 L CNN
-F 2 "" H 3238 3400 50  0001 C CNN
+F 2 "Capacitor_THT:CP_Axial_L42.5mm_D20.0mm_P49.00mm_Horizontal" H 3238 3400 50  0001 C CNN
 F 3 "~" H 3200 3550 50  0001 C CNN
 	1    3200 3550
@@
 F 0 "C4" H 3718 3596 50  0000 L CNN
 F 1 "2µ2 tant" H 3650 3675 50  0000 L CNN
-F 2 "" H 3638 3400 50  0001 C CNN
+F 2 "Capacitor_THT:CP_Axial_L11.0mm_D5.0mm_P18.00mm_Horizontal" H 3638 3400 50  0001 C CNN
 F 3 "~" H 3600 3550 50  0001 C CNN
 	1    3600 3550
@@
 F 0 "C6" H 4668 3596 50  0000 L CNN
 F 1 "1µ" H 4668 3505 50  0000 L CNN
-F 2 "" H 4588 3400 50  0001 C CNN
+F 2 "Capacitor_THT:CP_Axial_L11.0mm_D5.0mm_P18.00mm_Horizontal" H 4588 3400 50  0001 C CNN
 F 3 "~" H 4550 3550 50  0001 C CNN
 	1    4550 3550
@@
 F 0 "C7" H 5568 2746 50  0000 L CNN
 F 1 "22µ tant" H 5568 2655 50  0000 L CNN
-F 2 "" H 5488 2550 50  0001 C CNN
+F 2 "Capacitor_THT:CP_Radial_Tantal_D6.0mm_P5.00mm" H 5488 2550 50  0001 C CNN
 F 3 "~" H 5450 2700 50  0001 C CNN
 	1    5450 2700
@@
 F 0 "U3" H 6000 2742 50  0000 C CNN
 F 1 "L7805" H 6000 2651 50  0000 C CNN
-F 2 "" H 6025 2350 50  0001 L CIN
+F 2 "Package_TO_SOT_THT:TO-220-3_Vertical" H 6025 2350 50  0001 L CIN
 F 3 "http://www.st.com/content/ccc/resource/technical/document/datasheet/41/4f/b3/b0/12/d4/47/88/CD00000444.pdf/files/CD00000444.pdf/jcr:content/translations/en.CD00000444.pdf" H 6000 2450 50  0001 C CNN
 	1    6000 2500
@@
 F 0 "U1" H 4100 3142 50  0000 C CNN
 F 1 "L7812" H 4100 3051 50  0000 C CNN
-F 2 "" H 4125 2750 50  0001 L CIN
+F 2 "Package_TO_SOT_THT:TO-220-3_Vertical" H 4125 2750 50  0001 L CIN
 F 3 "http://www.st.com/content/ccc/resource/technical/document/datasheet/41/4f/b3/b0/12/d4/47/88/CD00000444.pdf/files/CD00000444.pdf/jcr:content/translations/en.CD00000444.pdf" H 4100 2850 50  0001 C CNN
 	1    4100 2900
@@
 F 0 "U2" H 4100 3600 50  0000 C CNN
 F 1 "L7912" H 4100 3509 50  0000 C CNN
-F 2 "" H 4100 3550 50  0001 C CIN
+F 2 "Package_TO_SOT_THT:TO-220-3_Vertical" H 4100 3550 50  0001 C CIN
 F 3 "http://www.st.com/content/ccc/resource/technical/document/datasheet/c9/16/86/41/c7/2b/45/f2/CD00000450.pdf/files/CD00000450.pdf/jcr:content/translations/en.CD00000450.pdf" H 4100 3750 50  0001 C CNN
 	1    4100 3750
@@
 F 0 "R1" V 1875 3000 50  0000 C CNN
 F 1 "0Ω1" V 1775 3000 50  0000 C CNN
-F 2 "" V 1705 3000 50  0001 C CNN
+F 2 "Package_TO_SOT_THT:TO-126-2_Vertical" V 1705 3000 50  0001 C CNN
 F 3 "~" H 1775 3000 50  0001 C CNN
 	1    1775 3000
@@
 F 0 "D5" V 4904 3629 50  0000 L CNN
 F 1 "BYV10" V 4995 3629 50  0000 L CNN
-F 2 "" H 4950 3550 50  0001 C CNN
+F 2 "Diode_THT:D_A-405_P7.62mm_Horizontal" H 4950 3550 50  0001 C CNN
 F 3 "~" H 4950 3550 50  0001 C CNN
 	1    4950 3550
@@
 F 0 "D4" V 4904 3179 50  0000 L CNN
 F 1 "BYV10" V 4995 3179 50  0000 L CNN
-F 2 "" H 4950 3100 50  0001 C CNN
+F 2 "Diode_THT:D_A-405_P7.62mm_Horizontal" H 4950 3100 50  0001 C CNN
 F 3 "~" H 4950 3100 50  0001 C CNN
 	1    4950 3100
@@
 F 0 "D3" V 4904 2779 50  0000 L CNN
 F 1 "1N4001" V 4995 2779 50  0000 L CNN
-F 2 "" H 4950 2700 50  0001 C CNN
+F 2 "Diode_THT:D_A-405_P10.16mm_Horizontal" H 4950 2700 50  0001 C CNN
 F 3 "~" H 4950 2700 50  0001 C CNN
 	1    4950 2700
@@
 F 0 "J2" H 7029 2992 50  0000 L CNN
 F 1 "12/5/0/-12VDC" H 7029 2901 50  0000 L CNN
-F 2 "" H 6950 3000 50  0001 C CNN
+F 2 "TerminalBlock:TerminalBlock_bornier-4_P5.08mm" H 6950 3000 50  0001 C CNN
 F 3 "~" H 6950 3000 50  0001 C CNN
 	1    6950 3000

Commit message: WIP: PCB fiddling.
Parts:
- removed R1: 0Ω1, Package_TO_SOT_THT:TO-126-2_Vertical, symbol Device:R
- D1: footprint Diode_THT:Diode_Bridge_Vishay_KBU -> Diode_THT:Diode_Bridge_32.0x5.6x17.0mm_P10.0mm_P7.5mm
- J2: value 12/5/0/-12VDC -> 5/12/0/-12VDC
Connections:
- net labels added: +12V, +5V, -12V, GND
- wire segments 68 -> 69
Changed lines of the file:
@@
 F 0 "D1" H 2500 3025 50  0000 L CNN
 F 1 "-AA+" H 2225 3225 50  0000 L CNN
-F 2 "Diode_THT:Diode_Bridge_Vishay_KBU" H 2350 3200 50  0001 C CNN
+F 2 "Diode_THT:Diode_Bridge_32.0x5.6x17.0mm_P10.0mm_P7.5mm" H 2350 3200 50  0001 C CNN
 F 3 "~" H 2350 3200 50  0001 C CNN
 	1    2350 3200
@@
 $EndComp
 $Comp
-L Device:R R1
-U 1 1 5C3A8191
-P 1775 3000
-F 0 "R1" V 1875 3000 50  0000 C CNN
-F 1 "0Ω1" V 1775 3000 50  0000 C CNN
-F 2 "Package_TO_SOT_THT:TO-126-2_Vertical" V 1705 3000 50  0001 C CNN
-F 3 "~" H 1775 3000 50  0001 C CNN
-	1    1775 3000
-	0    1    1    0
-$EndComp
-$Comp
 L Device:D_Schottky D5
 U 1 1 5C3A82BE
@@
 	1600 3100 1600 3500
 Wire Wire Line
-	1600 3000 1625 3000
-Wire Wire Line
 	2650 3200 2650 2900
 Wire Wire Line
@@
 Wire Wire Line
 	3200 3400 3200 3325
-Wire Wire Line
-	1925 3000 1950 3000
 Wire Wire Line
 	1950 3000 1950 3325
@@
 P 6950 3000
 F 0 "J2" H 7029 2992 50  0000 L CNN
-F 1 "12/5/0/-12VDC" H 7029 2901 50  0000 L CNN
+F 1 "5/12/0/-12VDC" H 7029 2901 50  0000 L CNN
 F 2 "TerminalBlock:TerminalBlock_bornier-4_P5.08mm" H 6950 3000 50  0001 C CNN
 F 3 "~" H 6950 3000 50  0001 C CNN
@@
 $EndComp
 Wire Wire Line
-	4950 2900 6750 2900
-Wire Wire Line
 	4950 3750 6750 3750
 Wire Wire Line
@@
 Wire Wire Line
 	6450 2500 6650 2500
-Wire Wire Line
-	6650 2500 6650 3000
-Wire Wire Line
-	6650 3000 6750 3000
 Connection ~ 6450 2500
 Wire Wire Line
@@
 	1    0    0    -1
 $EndComp
+Text Label 1950 3000 0    50   ~ 0
+GND
+Text Label 4550 2900 0    50   ~ 0
++12V
+Text Label 4550 3750 0    50   ~ 0
+-12V
+Text Label 6450 2500 0    50   ~ 0
++5V
+Wire Wire Line
+	1600 3000 1950 3000
+Wire Wire Line
+	6650 2500 6650 2900
+Wire Wire Line
+	6650 2900 6750 2900
+Wire Wire Line
+	4950 2900 6550 2900
+Wire Wire Line
+	6550 2900 6550 3000
+Wire Wire Line
+	6550 3000 6750 3000
 $EndSCHEMATC
